File: kicad/FASTUSBaspAdapter.kicad_pcb (KiCad board)
At the start: 2 copper layers, 71.1 x 29.2 mm, 2 parts, among them J1 CONN_01X06, U1 stm32f103c8t6-module-china

Commit message: improve the design little bit
Connections:
- U1 pad 19: Net-(U1-Pad19) -> /GND
- U1 pad 20: Net-(U1-Pad20) -> /Vcc_3.3v
- U1 pad 38: /Vcc_3.3v -> Net-(U1-Pad38)
- U1 pad 39: /GND -> Net-(U1-Pad39)
Routing:
- net /Vcc_3.3v: track 61.9 -> 15.4 mm
- net /RST: track 70.4 -> 56.7 mm
